Commit message: update

File: urdf/zumo32u4.urdf (robot description, URDF)
Before this commit: robot zumo32u4, 3 links, 2 joints
Links:
- added link map
- added link odom
Joints:
- added joint jointbaselink: type planar, parent map, child base_link, origin xyz=0 0 0 rpy=0 0 0, axis 0 0 1
- added joint jointodom: type fixed, parent base_link, child odom, origin xyz=0 0 0 rpy=0 0 0

Commit message: update

File: urdf/zumo32u4.urdf (robot description, URDF)
Before this commit: robot zumo32u4, 5 links, 4 joints
Joints:
- joint jointbaselink: type planar -> fixed

Commit message: update

File: urdf/zumo32u4.urdf (robot description, URDF)
Before this commit: robot zumo32u4, 1 links, 0 joints
Links:
- link base_link: geometry visual mesh filename=package://cartographer_ros/urdf/zumo32u4.STL scale=1 1 1
